File: main_board_8P3/main_board_8P3.kicad_pcb (KiCad board)
At the start: 2 copper layers, 114.3 x 86.4 mm, 47 parts

Commit message: Спроектированы варианты основных плат для МК в корпусах 8P3 и 8S2. Повторно выбраны значения свойсва Placement Type футпринтов
Parts:
- DD1: value IC_MCU_AVR_TINY_25-45-85_S8S1 -> IC_MCU_AVR_TINY_25-45-85_8P3; footprint KCL:P-SO-08 -> KCL:P-DIP-08
Routing:
- net /PB5: track 208.8 -> 203.7 mm, vias 3 -> 2
- net /VCC: track 27.2 -> 24.1 mm
- net /PB4: track 218.7 -> 221.7 mm
- net /PB3: track 246.9 -> 249.9 mm
- net COM: track 401.2 -> 399.2 mm
- net /PB2: track 189.5 -> 188.0 mm
- net /PB1: track 206.4 -> 205.4 mm
Other:
- board text added: "8P3"
- board text removed: "S8S1"

Commit message: Обновлены УГО ИМС
Parts:
- removed DD1: IC_MCU_AVR_TINY_25-45-85_8P3, KCL:P-DIP-08
- added D1: ATtiny25-20PU, KCL:P-DIP-08, F.Cu at (148.6, 104.1)
Changed lines of the file:
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@@
-(kicad_pcb (version 20171130) (host pcbnew 5.0.0-fee4fd1~66~ubuntu18.04.1)
+(kicad_pcb (version 20171130) (host pcbnew 5.0.2-bee76a0~70~ubuntu18.04.1)
   (general
     (thickness 1.5)
@@
   (title_block
     (title main_board_8P3)
-    (date 2019-02-18)
+    (date 2019-05-15)
     (rev 1)
     (company "Igor Vladimirovich Ivanov")
@@
     (pad_drill 0.762)
     (pad_to_mask_clearance 0.2)
+    (solder_mask_min_width 0.25)
     (aux_axis_origin 0 0)
     (visible_elements 7FFFFFFF)
@@
   (module KCL:P-DIP-08 (layer F.Cu)
     (at 148.59 104.14)
-    (fp_text reference DD1 (at 0 -5.715) (layer F.SilkS)
-      (effects (font (size 1 1) (thickness 0.2)))
-    )
-    (fp_text value IC_MCU_AVR_TINY_25-45-85_8P3 (at 0 -7.62) (layer F.Fab) hide
+    (fp_text reference D1 (at 0 -5.715) (layer F.SilkS)
+      (effects (font (size 1 1) (thickness 0.2)))
+    )
+    (fp_text value ATtiny25-20PU (at 0 -6.985) (layer F.Fab) hide
       (effects (font (size 1 1) (thickness 0.2)))
     )
@@
       (net 2 "Net-(C2-Pad1)"))
   )
-  (gr_text 8P3 (at 158.75 109.22) (layer F.SilkS)
+  (gr_text 8P3 (at 158.75 104.14) (layer F.SilkS)
     (effects (font (size 3 3) (thickness 0.6)))
   )
@@
   (gr_line (start 205.74 60.96) (end 205.74 147.32) (angle 90) (layer Edge.Cuts) (width 0.4))
   (gr_line (start 91.44 60.96) (end 205.74 60.96) (angle 90) (layer Edge.Cuts) (width 0.4))
-  (gr_text ATtiny25/45/85 (at 172.72 104.14) (layer F.SilkS)
+  (gr_text ATtiny25/45/85 (at 124.46 104.14) (layer F.SilkS)
     (effects (font (size 3 3) (thickness 0.6)))
   )
@@
   (segment (start 151.13 142.24) (end 175.26 118.11) (width 0.6) (layer F.Cu) (net 6))
   (segment (start 175.26 92.075) (end 175.26 74.93) (width 0.6) (layer B.Cu) (net 6))
-  (via (at 175.26 92.075) (size 2) (drill 0.5) (layers F.Cu B.Cu) (net 6) (status 1000000))
+  (via (at 175.26 92.075) (size 2) (drill 0.5) (layers F.Cu B.Cu) (net 6))
   (segment (start 175.26 98.425) (end 175.26 92.075) (width 0.6) (layer B.Cu) (net 6))
   (via (at 175.26 98.425) (size 2) (drill 0.5) (layers F.Cu B.Cu) (net 6))
