File: main_board_8P3/main_board_8P3.kicad_pcb (KiCad board)
At the start: 2 copper layers, 114.3 x 86.4 mm, 47 parts

Commit message: Отредактированы чертежи плат (обновлён ФП разъёма питания, удалено отчество в основной надписи)
Parts:
- XP2: value CONNECTOR_M_BARREL_20_POWER -> CONNECTOR_M_BARREL_SW
Changed lines of the file:
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@@
-(kicad_pcb (version 20171130) (host pcbnew 5.1.4)
+(kicad_pcb (version 20171130) (host pcbnew 5.1.5-52549c5~84~ubuntu19.10.1)
   (general
     (thickness 1.5)
@@
   (title_block
     (title main_board_8P3)
-    (date 2019-11-04)
+    (date 2020-03-05)
     (rev 1)
-    (company "Igor Vladimirovich Ivanov")
+    (company "Igor Ivanov")
     (comment 1 https://github.com/Adept666)
     (comment 2 "This project is licensed under GNU General Public License v3.0 or later")
@@
       (effects (font (size 1 1) (thickness 0.2)))
     )
-    (fp_text value CONNECTOR_M_BARREL_20_POWER (at 0 24.765 180) (layer F.Fab) hide
+    (fp_text value CONNECTOR_M_BARREL_SW (at 0 21.59 180) (layer F.Fab) hide
       (effects (font (size 1 1) (thickness 0.2)))
     )
@@
     (fp_line (start 4.5 1.651) (end 4.5 3) (layer F.SilkS) (width 0.2))
     (fp_line (start 4.5 -3.7) (end 4.5 -1.651) (layer F.SilkS) (width 0.2))
-    (pad 2 thru_hole rect (at 0 3 90) (size 5 3) (drill oval 3 0.7) (layers B.Cu B.Mask)
-      (net 35 "Net-(SA2-PadCOM1)"))
-    (pad 3 thru_hole rect (at 4.7 0 90) (size 3 5) (drill oval 0.7 3) (layers B.Cu B.Mask))
-    (pad 1 thru_hole rect (at 0 -3 90) (size 5 3) (drill oval 3.5 0.7) (layers B.Cu B.Mask)
-      (net 36 "Net-(SA2-PadCOM2)"))
+    (pad S thru_hole rect (at 0 3 90) (size 5 3) (drill oval 3 0.7) (layers B.Cu B.Mask))
+    (pad SN thru_hole rect (at 4.7 0 90) (size 3 5) (drill oval 0.7 3) (layers B.Cu B.Mask))
+    (pad C thru_hole rect (at 0 -3 90) (size 5 3) (drill oval 3.5 0.7) (layers B.Cu B.Mask))
   )
   (module KCL:VMH-STA-DA5 (layer F.Cu)
