File: main_board_S8S1/main_board_S8S1.sch (KiCad schematic (older format))
At the start: 47 parts

Commit message: Подписаны разъёмы, переключатели, светодиоды и ИМС. Скрыты имена футпринтов. Показана мощность резисторов. Свойства текстовых полей УГО приведены к единообразию
Parts:
- DD1: Title (none) -> ATtiny25/45/85 S8S1
- HL1, SA1, XS1: Title (none) -> CRYSTAL
- HL2, SA2, XP2, XS2: Title (none) -> POWER
- HL3: Title (none) -> PB0
- HL4: Title (none) -> PB1
- HL5: Title (none) -> PB2
- HL6: Title (none) -> PB3
- HL7: Title (none) -> PB4
- R1, R10, R11, R12, R13, R2, R3, R4, R5, R6, R7, R8, R9: Power (none) -> 0,125 Вт
- SA3: Title (none) -> PB0...4
- SB1: Title (none) -> RESET
- XP1, XP4: Title (none) -> DATA
- XP3: Title (none) -> PROG

Commit message: Свойства текстовых полей составных частей УГО ключа SA3 приведены к единообразию
Parts:
- SA3: Title PB0...4 -> (none)
Changed lines of the file:
@@
 EESchema Schematic File Version 4
-LIBS:main_board_S8S1-cache
 EELAYER 26 0
 EELAYER END
@@
 U 1 1 5AD54C53
 P 9500 2400
-F 0 "SA3" H 9500 3050 100 0000 C CNN
+F 0 "SA3" H 9500 3100 100 0000 C CNN
 F 1 "SWITCH_BLOCK_05" H 9500 2400 100 0001 C CNN
 F 2 "KCL:SW-NDI(R)-05" H 9500 2400 60  0001 C CNN
 F 3 "" H 9500 2400 60  0001 C CNN
-F 4 "PB0...4" H 9500 2900 100 0000 C CNN "Title"
-F 5 "NDI-05H-V" H 9500 2750 60  0000 C CNN "Product"
-F 6 "Diptronics" H 9500 2650 60  0000 C CNN "Manufacturer"
+F 4 "PB0...4" H 9500 2950 100 0000 C CNN "Title"
+F 5 "NDI-05H-V" H 9500 2800 60  0000 C CNN "Product"
+F 6 "Diptronics" H 9500 2700 60  0000 C CNN "Manufacturer"
 	1    9500 2400
 	1    0    0    -1
@@
 P 9500 3900
 F 0 "SA3" H 9500 4200 100 0000 C CNN
-F 1 "SWITCH_BLOCK_05" H 9500 4350 100 0001 C CNN
-F 2 "KCL:SW-NDI(R)-05" H 9400 4690 60  0001 C CNN
-F 3 "" H 9400 4690 60  0001 C CNN
-F 4 "PB0...4" H 0   0   50  0001 C CNN "Title"
+F 1 "SWITCH_BLOCK_05" H 9500 3900 100 0001 C CNN
+F 2 "KCL:SW-NDI(R)-05" H 9500 3900 60  0001 C CNN
+F 3 "" H 9500 3900 60  0001 C CNN
 	2    9500 3900
 	1    0    0    -1
@@
 P 9500 5400
 F 0 "SA3" H 9500 5700 100 0000 C CNN
-F 1 "SWITCH_BLOCK_05" H 9500 5850 100 0001 C CNN
-F 2 "KCL:SW-NDI(R)-05" H 9400 6190 60  0001 C CNN
-F 3 "" H 9400 6190 60  0001 C CNN
-F 4 "PB0...4" H 0   0   50  0001 C CNN "Title"
+F 1 "SWITCH_BLOCK_05" H 9500 5400 100 0001 C CNN
+F 2 "KCL:SW-NDI(R)-05" H 9500 5400 60  0001 C CNN
+F 3 "" H 9500 5400 60  0001 C CNN
 	3    9500 5400
 	1    0    0    -1
@@
 P 9500 6900
 F 0 "SA3" H 9500 7200 100 0000 C CNN
-F 1 "SWITCH_BLOCK_05" H 9500 7350 100 0001 C CNN
-F 2 "KCL:SW-NDI(R)-05" H 9400 7690 60  0001 C CNN
-F 3 "" H 9400 7690 60  0001 C CNN
-F 4 "PB0...4" H 0   0   50  0001 C CNN "Title"
+F 1 "SWITCH_BLOCK_05" H 9500 6900 100 0001 C CNN
+F 2 "KCL:SW-NDI(R)-05" H 9500 6900 60  0001 C CNN
+F 3 "" H 9500 6900 60  0001 C CNN
 	4    9500 6900
 	1    0    0    -1
@@
 P 9500 8400
 F 0 "SA3" H 9500 8700 100 0000 C CNN
-F 1 "SWITCH_BLOCK_05" H 9500 8850 100 0001 C CNN
-F 2 "KCL:SW-NDI(R)-05" H 9400 9190 60  0001 C CNN
-F 3 "" H 9400 9190 60  0001 C CNN
-F 4 "PB0...4" H 0   0   50  0001 C CNN "Title"
+F 1 "SWITCH_BLOCK_05" H 9500 8400 100 0001 C CNN
+F 2 "KCL:SW-NDI(R)-05" H 9500 8400 60  0001 C CNN
+F 3 "" H 9500 8400 60  0001 C CNN
 	5    9500 8400
 	1    0    0    -1

Commit message: Отредактирована библиотека проекта. Обновлена схема и плата
Parts:
- XP1, XP4: symbol main_board_S8S1:CONNECTOR_M_014_20_ДАННЫЕ -> main_board_S8S1:CONNECTOR_M_014_20_DATA
- XP2: symbol main_board_S8S1:CONNECTOR_M_BARREL_20_ПИТАНИЕ -> main_board_S8S1:CONNECTOR_M_BARREL_20_POWER
- XP3: symbol main_board_S8S1:CONNECTOR_M_010_20_ПРОГРАММАТОР -> main_board_S8S1:CONNECTOR_M_010_20_PROG
- XS1: symbol main_board_S8S1:CONNECTOR_F_002_20_КВАРЦ -> main_board_S8S1:CONNECTOR_F_002_20_CRYSTAL
- XS2: symbol main_board_S8S1:CONNECTOR_F_002_20_ПИТАНИЕ -> main_board_S8S1:CONNECTOR_F_002_20_POWER
Changed lines of the file:
@@
 	4600 6450 4650 6450
 $Comp
-L main_board_S8S1:CONNECTOR_M_014_20_ДАННЫЕ XP4
+L main_board_S8S1:CONNECTOR_M_014_20_DATA XP4
 U 1 1 5AD7D10B
 P 14000 1900
@@
 $EndComp
 $Comp
-L main_board_S8S1:CONNECTOR_M_010_20_ПРОГРАММАТОР XP3
+L main_board_S8S1:CONNECTOR_M_010_20_PROG XP3
 U 1 1 5AD7D48C
 P 5500 1900
@@
 $EndComp
 $Comp
-L main_board_S8S1:CONNECTOR_F_002_20_КВАРЦ XS1
+L main_board_S8S1:CONNECTOR_F_002_20_CRYSTAL XS1
 U 1 1 5AD7D71D
 P 3000 6400
@@
 $EndComp
 $Comp
-L main_board_S8S1:CONNECTOR_F_002_20_ПИТАНИЕ XS2
+L main_board_S8S1:CONNECTOR_F_002_20_POWER XS2
 U 1 1 5AD7D7C6
 P 3000 10500
@@
 $EndComp
 $Comp
-L main_board_S8S1:CONNECTOR_M_BARREL_20_ПИТАНИЕ XP2
+L main_board_S8S1:CONNECTOR_M_BARREL_20_POWER XP2
 U 1 1 5AD7D885
 P 3000 8750
@@
 $EndComp
 $Comp
-L main_board_S8S1:CONNECTOR_M_014_20_ДАННЫЕ XP1
+L main_board_S8S1:CONNECTOR_M_014_20_DATA XP1
 U 1 1 5AD7E6B0
 P 3000 1900

Commit message: Применены собственные символы общей точки и питания. Завершено обновление схемы после дорабоки бибиотеки проекта
Parts:
- XP1, XP4: value CONNECTOR_M_014_20_ДАННЫЕ -> CONNECTOR_M_014_20_DATA
- XP2: value CONNECTOR_M_BARREL_20_ПИТАНИЕ -> CONNECTOR_M_BARREL_20_POWER
- XP3: value CONNECTOR_M_010_20_ПРОГРАММАТОР -> CONNECTOR_M_010_20_PROG
- XS1: value CONNECTOR_F_002_20_КВАРЦ -> CONNECTOR_F_002_20_CRYSTAL
- XS2: value CONNECTOR_F_002_20_ПИТАНИЕ -> CONNECTOR_F_002_20_POWER
Connections:
- net labels added: POWER_COM, POWER_V
- net labels removed: +5V, GND
- wire segments 187 -> 189

Commit message: Обновлены УГО ИМС
Parts:
- D1: renamed from DD1; value IC_MCU_AVR_TINY_25-45-85_S8S1 -> ATtiny25-20SSU; symbol KCL:IC_MCU_AVR_TINY_25-45-85_S8S1 -> ICL_MICROCHIP:ATtiny25-20SSU
Changed lines of the file:
@@
 Sheet 1 1
 Title "main_board_S8S1"
-Date "2019-02-17"
+Date "2019-05-15"
 Rev "2"
 Comp "Igor Vladimirovich Ivanov"
@@
 Text Label 6200 3900 2    70   ~ 0
 PB1
-Wire Bus Line
-	3750 750  13250 750
 Wire Wire Line
 	13750 1650 13750 1900
@@
 	8750 750  8750 7150
 Wire Bus Line
-	6500 2400 6500 750
-Wire Wire Line
-	6750 2900 6750 2650
+	6750 2400 6750 750
+Wire Wire Line
+	7000 2900 7000 2650
 Text Label 8700 2650 2    70   ~ 0
 PB0
@@
 	8750 2400 8500 2400
 Wire Wire Line
-	6500 1900 6750 1900
-Wire Wire Line
-	6500 2150 6750 2150
-Wire Wire Line
-	6500 2400 6750 2400
+	6750 1900 7000 1900
+Wire Wire Line
+	6750 2150 7000 2150
+Wire Wire Line
+	6750 2400 7000 2400
 Text Label 8700 2400 2    70   ~ 0
 PB1
@@
 Text Label 8700 1900 2    70   ~ 0
 VCC
-Text Label 6550 2150 0    70   ~ 0
+Text Label 6800 2150 0    70   ~ 0
 PB3
-Text Label 6550 2400 0    70   ~ 0
+Text Label 6800 2400 0    70   ~ 0
 PB4
-Text Label 6550 1900 0    70   ~ 0
+Text Label 6800 1900 0    70   ~ 0
 PB5
 Wire Wire Line
@@
 	7500 7150 8000 7150
 $Comp
-L KCL:IC_MCU_AVR_TINY_25-45-85_S8S1 DD1
+L ICL_MICROCHIP:ATtiny25-20SSU D1
 U 1 1 5B6FE9DE
-P 7625 1900
-F 0 "DD1" H 7625 2500 100 0000 C CNN
-F 1 "IC_MCU_AVR_TINY_25-45-85_S8S1" H 7625 1900 100 0001 C CNN
-F 2 "KCL:P-SO-08" H 7625 1900 60  0001 C CNN
-F 3 "" H 7625 1900 60  0001 C CNN
-F 4 "ATtiny25/45/85 S8S1" H 7625 2350 100 0000 C CNN "Title"
-F 5 "ATtiny25/45/85" H 7625 2200 60  0000 C CNN "Product"
-F 6 "Microchip" H 7625 2100 60  0000 C CNN "Manufacturer"
-	1    7625 1900
+P 7750 1900
+F 0 "D1" H 7750 2500 100 0000 C CNN
+F 1 "ATtiny25-20SSU" H 7750 1900 100 0001 C CNN
+F 2 "KCL:P-SO-08" H 7750 1900 60  0001 C CNN
+F 3 "http://ww1.microchip.com/downloads/en/DeviceDoc/Atmel-2586-AVR-8-bit-Microcontroller-ATtiny25-ATtiny45-ATtiny85_Datasheet.pdf" H 7750 1900 60  0001 C CNN
+F 4 "ATtiny25/45/85 S8S1" H 7750 2350 100 0000 C CNN "Title"
+F 5 "ATtiny25/45/85" H 7750 2200 60  0000 C CNN "Product"
+F 6 "Microchip" H 7750 2100 60  0000 C CNN "Manufacturer"
+	1    7750 1900
 	1    0    0    -1
 $EndComp
@@
 L KCL:POWER_COM #PWR0112
 U 1 1 5C7FE3E0
-P 6750 2900
-F 0 "#PWR0112" H 6750 2900 100 0001 C CNN
-F 1 "POWER_COM" H 6750 2900 100 0001 C CNN
-F 2 "" H 6750 2900 60  0001 C CNN
-F 3 "" H 6750 2900 60  0001 C CNN
-F 4 "COM" H 6750 2900 100 0001 C CNN "Label"
-	1    6750 2900
+P 7000 2900
+F 0 "#PWR0112" H 7000 2900 100 0001 C CNN
+F 1 "POWER_COM" H 7000 2900 100 0001 C CNN
+F 2 "" H 7000 2900 60  0001 C CNN
+F 3 "" H 7000 2900 60  0001 C CNN
+F 4 "COM" H 7000 2900 100 0001 C CNN "Label"
+	1    7000 2900
 	1    0    0    -1
 $EndComp
@@
 	1    0    0    -1
 $EndComp
+Wire Bus Line
+	3750 750  13250 750
 $EndSCHEMATC
