File: main_board_S8S1/main_board_S8S1.sch (KiCad schematic (older format))
At the start: 47 parts

Commit message: Схемы и платы обновлены в связи с переименованием футпринта стойки VMH-STA-DA5
Parts:
- VMH1, VMH2, VMH3, VMH4: footprint KCL:STA-DA5 -> KCL:VMH-STA-DA5
Changed lines of the file:
@@
 EESchema Schematic File Version 4
 LIBS:main_board_S8S1-cache
-EELAYER 29 0
+EELAYER 30 0
 EELAYER END
 $Descr A3 16535 11693
@@
 Sheet 1 1
 Title "main_board_S8S1"
-Date "2019-07-12"
+Date "2019-09-04"
 Rev "2"
 Comp "Igor Vladimirovich Ivanov"
@@
 F 0 "VMH1" H 14500 6800 100 0000 C CNN
 F 1 "VIRTUAL_MOUNTING-HOLE" H 14500 6400 100 0001 C CNN
-F 2 "KCL:STA-DA5" H 14500 6400 60  0001 C CNN
+F 2 "KCL:VMH-STA-DA5" H 14500 6400 60  0001 C CNN
 F 3 "" H 14500 6400 60  0001 C CNN
 F 4 "Нижняя стойка: DI5M3x08 (Vogt)" H 14500 6700 60  0000 C CNN "Нижняя стойка"
@@
 F 0 "VMH2" H 14500 7800 100 0000 C CNN
 F 1 "VIRTUAL_MOUNTING-HOLE" H 14500 7400 100 0001 C CNN
-F 2 "KCL:STA-DA5" H 14500 7400 60  0001 C CNN
+F 2 "KCL:VMH-STA-DA5" H 14500 7400 60  0001 C CNN
 F 3 "" H 14500 7400 60  0001 C CNN
 F 4 "Нижняя стойка: DI5M3x08 (Vogt)" H 14500 7700 60  0000 C CNN "Нижняя стойка"
@@
 F 0 "VMH3" H 14500 8800 100 0000 C CNN
 F 1 "VIRTUAL_MOUNTING-HOLE" H 14500 8400 100 0001 C CNN
-F 2 "KCL:STA-DA5" H 14500 8400 60  0001 C CNN
+F 2 "KCL:VMH-STA-DA5" H 14500 8400 60  0001 C CNN
 F 3 "" H 14500 8400 60  0001 C CNN
 F 4 "Нижняя стойка: DI5M3x08 (Vogt)" H 14500 8700 60  0000 C CNN "Нижняя стойка"
@@
 F 0 "VMH4" H 14500 9800 100 0000 C CNN
 F 1 "VIRTUAL_MOUNTING-HOLE" H 14500 9400 100 0001 C CNN
-F 2 "KCL:STA-DA5" H 14500 9400 60  0001 C CNN
+F 2 "KCL:VMH-STA-DA5" H 14500 9400 60  0001 C CNN
 F 3 "" H 14500 9400 60  0001 C CNN
 F 4 "Нижняя стойка: DI5M3x08 (Vogt)" H 14500 9700 60  0000 C CNN "Нижняя стойка"

Commit message: Схемы скорректированы с учётом изменений в УГО переключателей
Parts:
- SA1, SA2: value SWITCH_SPECIAL_SK-42D01-G -> SWITCH_GENERAL_04P_02T; symbol KCL:SWITCH_SPECIAL_SK-42D01-G -> KCL:SWITCH_GENERAL_04P_02T
- SA3: value SWITCH_BLOCK_05 -> SWITCH_GENERAL_01P_01T_NO_05U; symbol KCL:SWITCH_BLOCK_05 -> KCL:SWITCH_GENERAL_01P_01T_NO_05U
- SB1: value SWITCH_BUTTON_NO_01 -> SWITCH_BUTTON_NON-LOCK_01P_01T_NO; symbol KCL:SWITCH_BUTTON_NO_01 -> KCL:SWITCH_BUTTON_NON-LOCK_01P_01T_NO
Changed lines of the file:
@@
 $EndDescr
 $Comp
-L KCL:SWITCH_SPECIAL_SK-42D01-G SA2
+L KCL:SWITCH_GENERAL_04P_02T SA2
 U 1 1 5AD54932
 P 4250 8500
 F 0 "SA2" H 4250 9150 100 0000 C CNN
-F 1 "SWITCH_SPECIAL_SK-42D01-G" H 4250 8500 100 0001 C CNN
+F 1 "SWITCH_GENERAL_04P_02T" H 4250 8500 100 0001 C CNN
 F 2 "KCL:SW-SK-42D01-G" H 4250 8500 60  0001 C CNN
 F 3 "" H 4250 8500 60  0001 C CNN
@@
 $EndComp
 $Comp
-L KCL:SWITCH_BUTTON_NO_01 SB1
+L KCL:SWITCH_BUTTON_NON-LOCK_01P_01T_NO SB1
 U 1 1 5AD5497D
 P 6750 7650
 F 0 "SB1" V 6950 7600 100 0000 R CNN
-F 1 "SWITCH_BUTTON_NO_01" V 6750 7650 100 0001 R CNN
+F 1 "SWITCH_BUTTON_NON-LOCK_01P_01T_NO" V 6750 7650 100 0001 R CNN
 F 2 "KCL:SW-07125" V 6750 7650 60  0001 R CNN
 F 3 "" V 6750 7650 60  0001 R CNN
@@
 $EndComp
 $Comp
-L KCL:SWITCH_BLOCK_05 SA3
+L KCL:SWITCH_GENERAL_01P_01T_NO_05U SA3
 U 1 1 5AD54C53
 P 9500 2400
 F 0 "SA3" H 9500 3100 100 0000 C CNN
-F 1 "SWITCH_BLOCK_05" H 9500 2400 100 0001 C CNN
+F 1 "SWITCH_GENERAL_01P_01T_NO_05U" H 9500 2400 100 0001 C CNN
 F 2 "KCL:SW-NDI(R)-05" H 9500 2400 60  0001 C CNN
 F 3 "" H 9500 2400 60  0001 C CNN
@@
 $EndComp
 $Comp
-L KCL:SWITCH_BLOCK_05 SA3
+L KCL:SWITCH_GENERAL_01P_01T_NO_05U SA3
 U 2 1 5AD54CB6
 P 9500 3900
 F 0 "SA3" H 9500 4200 100 0000 C CNN
-F 1 "SWITCH_BLOCK_05" H 9500 3900 100 0001 C CNN
+F 1 "SWITCH_GENERAL_01P_01T_NO_05U" H 9500 3900 100 0001 C CNN
 F 2 "KCL:SW-NDI(R)-05" H 9500 3900 60  0001 C CNN
 F 3 "" H 9500 3900 60  0001 C CNN
@@
 $EndComp
 $Comp
-L KCL:SWITCH_BLOCK_05 SA3
+L KCL:SWITCH_GENERAL_01P_01T_NO_05U SA3
 U 3 1 5AD54CF3
 P 9500 5400
 F 0 "SA3" H 9500 5700 100 0000 C CNN
-F 1 "SWITCH_BLOCK_05" H 9500 5400 100 0001 C CNN
+F 1 "SWITCH_GENERAL_01P_01T_NO_05U" H 9500 5400 100 0001 C CNN
 F 2 "KCL:SW-NDI(R)-05" H 9500 5400 60  0001 C CNN
 F 3 "" H 9500 5400 60  0001 C CNN
@@
 $EndComp
 $Comp
-L KCL:SWITCH_BLOCK_05 SA3
+L KCL:SWITCH_GENERAL_01P_01T_NO_05U SA3
 U 4 1 5AD54D26
 P 9500 6900
 F 0 "SA3" H 9500 7200 100 0000 C CNN
-F 1 "SWITCH_BLOCK_05" H 9500 6900 100 0001 C CNN
+F 1 "SWITCH_GENERAL_01P_01T_NO_05U" H 9500 6900 100 0001 C CNN
 F 2 "KCL:SW-NDI(R)-05" H 9500 6900 60  0001 C CNN
 F 3 "" H 9500 6900 60  0001 C CNN
@@
 $EndComp
 $Comp
-L KCL:SWITCH_BLOCK_05 SA3
+L KCL:SWITCH_GENERAL_01P_01T_NO_05U SA3
 U 5 1 5AD54D57
 P 9500 8400
 F 0 "SA3" H 9500 8700 100 0000 C CNN
-F 1 "SWITCH_BLOCK_05" H 9500 8400 100 0001 C CNN
+F 1 "SWITCH_GENERAL_01P_01T_NO_05U" H 9500 8400 100 0001 C CNN
 F 2 "KCL:SW-NDI(R)-05" H 9500 8400 60  0001 C CNN
 F 3 "" H 9500 8400 60  0001 C CNN
@@
 $EndComp
 $Comp
-L KCL:SWITCH_SPECIAL_SK-42D01-G SA1
+L KCL:SWITCH_GENERAL_04P_02T SA1
 U 1 1 5AD7E9C3
 P 4250 5950
 F 0 "SA1" H 4250 6700 100 0000 C CNN
-F 1 "SWITCH_SPECIAL_SK-42D01-G" H 4250 5950 100 0001 C CNN
+F 1 "SWITCH_GENERAL_04P_02T" H 4250 5950 100 0001 C CNN
 F 2 "KCL:SW-SK-42D01-G" H 4250 5950 60  0001 C CNN
 F 3 "" H 4250 5950 60  0001 C CNN

Commit message: Платы обновлены в связи с переименованием футпринтов катушек индуктивности
Parts:
- L1: footprint KCL:L-SDR0805 -> KCL:I-SDR0805
Changed lines of the file:
@@
 Sheet 1 1
 Title "main_board_S8S1"
-Date "2019-09-04"
+Date "2019-11-04"
 Rev "2"
 Comp "Igor Vladimirovich Ivanov"
@@
 F 0 "L1" H 7250 4800 100 0000 C CNN
 F 1 "INDUCTOR_FMC" H 7250 4150 100 0001 C CNN
-F 2 "KCL:L-SDR0805" H 7250 4150 60  0001 C CNN
+F 2 "KCL:I-SDR0805" H 7250 4150 60  0001 C CNN
 F 3 "" H 7250 4150 60  0001 C CNN
 F 4 "47 мкГн" H 7250 4700 60  0000 C CNN "Inductance"

Commit message: Отредактированы схемы (заменено УГО разъёма питания, удалено отчество в основной надписи)
Parts:
- XP2: value CONNECTOR_M_BARREL_20_POWER -> CONNECTOR_M_BARREL_SW; symbol main_board_S8S1:CONNECTOR_M_BARREL_20_POWER -> KCL:CONNECTOR_M_BARREL_SW
Changed lines of the file:
@@
 EESchema Schematic File Version 4
-LIBS:main_board_S8S1-cache
 EELAYER 30 0
 EELAYER END
@@
 Sheet 1 1
 Title "main_board_S8S1"
-Date "2019-11-04"
+Date "2020-03-05"
 Rev "2"
-Comp "Igor Vladimirovich Ivanov"
+Comp "Igor Ivanov"
 Comment1 "https://github.com/Adept666"
 Comment2 "This project is licensed under GNU General Public License v3.0 or later"
@@
 $EndComp
 $Comp
-L main_board_S8S1:CONNECTOR_M_BARREL_20_POWER XP2
-U 1 1 5AD7D885
-P 3000 8750
-F 0 "XP2" H 3750 9600 100 0000 C CNN
-F 1 "CONNECTOR_M_BARREL_20_POWER" H 3000 8750 100 0001 C CNN
-F 2 "KCL:CON-PJ-002B" H 3000 8750 60  0001 C CNN
-F 3 "" H 3000 8750 60  0001 C CNN
-F 4 "POWER" H 3750 9450 100 0000 C CNN "Title"
-F 5 "PJ-002B" H 3750 9300 60  0000 C CNN "Product"
-F 6 "CUI" H 3750 9200 60  0000 C CNN "Manufacturer"
-	1    3000 8750
-	-1   0    0    -1
-$EndComp
-$Comp
 L main_board_S8S1:CONNECTOR_M_014_20_DATA XP1
 U 1 1 5AD7E6B0
@@
 Wire Bus Line
 	9000 750  13250 750
+$Comp
+L KCL:CONNECTOR_M_BARREL_SW XP2
+U 1 1 5AD7D885
+P 3000 8750
+F 0 "XP2" H 3250 9350 100 0000 C CNN
+F 1 "CONNECTOR_M_BARREL_SW" H 3000 8750 100 0001 C CNN
+F 2 "KCL:CON-PJ-002B" H 3000 8750 60  0001 C CNN
+F 3 "" H 3000 8750 60  0001 C CNN
+F 4 "POWER" H 3250 9200 100 0000 C CNN "Title"
+F 5 "PJ-002B" H 3250 9050 60  0000 C CNN "Product"
+F 6 "CUI" H 3250 8950 60  0000 C CNN "Manufacturer"
+	1    3000 8750
+	-1   0    0    -1
+$EndComp
 $EndSCHEMATC
